File: ICM-42670-P Breakout Board.kicad_sch (KiCad schematic)
At the start: 12 parts, among them J2 Conn_01x09_Pin, U1 ICM-42670-P, U2 MCP1700x-330xxTT

Commit message: Update LED PART
Parts:
- D1: Part (none) -> KT-0603R
Changed lines of the file:
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@@
+			)
+		)
+		(property "Part" "KT-0603R"
+			(at 210.82 62.23 0)
+			(effects
+				(font
+					(size 1.27 1.27)
+				)
+				(hide yes)
 			)
 		)

Commit message: Add JLCPCB Part#
Parts:
- C1: JLCPCB Part # (none) -> C1525
- C2, C4, C5: JLCPCB Part # (none) -> C12530; Specification X7R, 2.2 µF ±10% 16V -> X7R, 2.2 µF ±20% 6.3V
- C3: JLCPCB Part # (none) -> C15195
- D1: JLCPCB Part # (none) -> C2290; Part KT-0603R -> (none)
- R1, R2: JLCPCB Part # (none) -> C328298
- R3: JLCPCB Part # (none) -> C352482; Specification (none) -> ±1% 0.0625 W (1/16 W)
- U1: JLCPCB Part # (none) -> C3288646
- U2: JLCPCB Part # (none) -> C39051
Changed lines of the file:
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@@
 			)
 		)
-		(property "Part" "KT-0603R"
+		(property "JLCPCB Part #" "C2290"
 			(at 210.82 62.23 0)
 			(effects
@@
 			)
 		)
+		(property "JLCPCB Part #" "C328298"
+			(at 168.91 91.44 90)
+			(effects
+				(font
+					(size 1.27 1.27)
+				)
+				(hide yes)
+			)
+		)
 		(pin "2"
 		)
@@
 			)
 		)
-		(property "Specification" "X7R, 2.2 µF ±10% 16V"
+		(property "Specification" "X7R, 2.2 µF ±20% 6.3V"
 			(at 199.39 91.44 0)
+			(effects
+				(font
+					(size 1.27 1.27)
+				)
+				(hide yes)
+			)
+		)
+		(property "JLCPCB Part #" "C12530"
+			(at 199.39 91.44 90)
 			(effects
 				(font
@@
 			)
 		)
+		(property "JLCPCB Part #" "C39051"
+			(at 213.36 101.6 0)
+			(effects
+				(font
+					(size 1.27 1.27)
+				)
+				(hide yes)
+			)
+		)
 		(pin "1"
 		)
@@
 			)
 		)
+		(property "JLCPCB Part #" "C3288646"
+			(at 59.69 86.36 0)
+			(effects
+				(font
+					(size 1.27 1.27)
+				)
+				(hide yes)
+			)
+		)
 		(pin "1"
 		)
@@
 			)
 		)
+		(property "JLCPCB Part #" "C328298"
+			(at 48.26 101.6 90)
+			(effects
+				(font
+					(size 1.27 1.27)
+				)
+				(hide yes)
+			)
+		)
 		(pin "2"
 		)
@@
 		)
 		(property "Description" "Unpolarized capacitor"
+			(at 35.56 106.68 0)
+			(effects
+				(font
+					(size 1.27 1.27)
+				)
+				(hide yes)
+			)
+		)
+		(property "JLCPCB Part #" "C15195"
 			(at 35.56 106.68 0)
 			(effects
@@
 			)
 		)
-		(property "Specification" "X7R, 2.2 µF ±10% 16V"
+		(property "Specification" "X7R, 2.2 µF ±20% 6.3V"
 			(at 227.33 91.44 0)
+			(effects
+				(font
+					(size 1.27 1.27)
+				)
+				(hide yes)
+			)
+		)
+		(property "JLCPCB Part #" "C12530"
+			(at 227.33 91.44 90)
 			(effects
 				(font
@@
 			)
 		)
+		(property "JLCPCB Part #" "C1525"
+			(at 165.1 107.95 0)
+			(effects
+				(font
+					(size 1.27 1.27)
+				)
+				(hide yes)
+			)
+		)
 		(pin "1"
 		)
@@
 			)
 		)
+		(property "JLCPCB Part #" "C352482"
+			(at 220.98 62.23 90)
+			(effects
+				(font
+					(size 1.27 1.27)
+				)
+				(hide yes)
+			)
+		)
+		(property "Specification" "±1% 0.0625 W (1/16 W)"
+			(at 220.98 62.23 90)
+			(effects
+				(font
+					(size 1.27 1.27)
+				)
+				(hide yes)
+			)
+		)
 		(pin "1"
 		)
@@
 			)
 		)
-		(property "Specification" "X7R, 2.2 µF ±10% 16V"
+		(property "Specification" "X7R, 2.2 µF ±20% 6.3V"
 			(at 179.07 107.95 0)
 			(effects
+				(font
+					(size 1.27 1.27)
+				)
+				(hide yes)
+			)
+		)
+		(property "JLCPCB Part #" "C12530"
+			(at 179.07 107.95 0)
+			(effects

Commit message: Changed BOM
Bom Reflects General Parts now
Parts:
- J2: now fitted
Changed lines of the file:
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@@
 		(in_bom yes)
 		(on_board yes)
-		(dnp yes)
+		(dnp no)
 		(fields_autoplaced yes)
 		(property "Reference" "J2"

Commit message: Adjusted schematic Page
A
Parts:
- C1: Specification X7R, 0.1 µF ±10% >= 16V -> X7R, 0.1 µF ±10% 6.3V
- C2, C4, C5: Specification X7R, 2.2 µF ±20% 6.3V -> X7R, 2.2 µF ±10% 6.3V
- C3: Specification (none) -> X7R, 2.2 µF ±10% 6.3V
Other:
- moved on the sheet: C1, C2, C3, C4, C5, D1, J2, R1, R2, R3, U1, U2
