File: 0603 Parts/ICM-42670-P Breakout Board 0603.kicad_pcb (KiCad board)
At the start: 2 copper layers, 18 x 26.5 mm, 12 parts, among them J2 Conn_01x09_Pin, U1 ICM-42670-P, U3 MCP1700x-300xxTT

Commit message: Fix DRC errors
Parts:
- moved C3 2.77 mm to (70.0, 40.5)
- moved R2 1.75 mm to (70.0, 37.2)
- moved C5 1.25 mm to (63.8, 28.0)
- moved U3 0.50 mm to (67.0, 28.0)
Routing:
- net /3V3_Clean: track 38.3 -> 40.6 mm, vias 0 -> 2
- net /FSYNC: track 22.0 -> 20.7 mm
- net /5V / 3V3: track 7.39 -> 8.42 mm
- net GND: track 46.5 -> 47.5 mm

Commit message: add b.silkscreen text
Other:
- board text added: "SleepyPandas"
Changed lines of the file:
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@@
+			)
+		)
+		(fp_text user "${REFERENCE}"
+			(at 0 0 90)
+			(unlocked yes)
+			(layer "F.Fab")
+			(effects
+				(font
+					(size 1 1)
+					(thickness 0.15)
+				)
 			)
 		)
 		(fp_text user "*"
 			(at -0.9398 -1 90)
-			(layer "F.Fab")
-			(effects
-				(font
-					(size 1 1)
-					(thickness 0.15)
-				)
-			)
-		)
-		(fp_text user "${REFERENCE}"
-			(at 0 0 90)
 			(unlocked yes)
 			(layer "F.Fab")
@@
 		(sheetname "/")
 		(sheetfile "ICM-42670-P Breakout Board 0603.kicad_sch")
-		(attr through_hole)
+		(attr through_hole dnp)
 		(fp_line
 			(start 1.38 1.27)
@@
 			(drill 1)
 			(layers "*.Cu" "*.Mask")
-			(remove_unused_layers yes)
-			(keep_end_layers yes)
-			(zone_layer_connections)
+			(remove_unused_layers no)
 			(net 5 "/FSYNC")
 			(pinfunction "Pin_1")
@@
 			(drill 1)
 			(layers "*.Cu" "*.Mask")
-			(remove_unused_layers yes)
-			(keep_end_layers yes)
-			(zone_layer_connections)
+			(remove_unused_layers no)
 			(net 3 "/INT1")
 			(pinfunction "Pin_2")
@@
 			(drill 1)
 			(layers "*.Cu" "*.Mask")
-			(remove_unused_layers yes)
-			(keep_end_layers yes)
-			(zone_layer_connections)
+			(remove_unused_layers no)
 			(net 4 "/SDO")
 			(pinfunction "Pin_3")
@@
 			(drill 1)
 			(layers "*.Cu" "*.Mask")
-			(remove_unused_layers yes)
-			(keep_end_layers yes)
-			(zone_layer_connections)
+			(remove_unused_layers no)
 			(net 8 "/SDA")
 			(pinfunction "Pin_4")
@@
 			(drill 1)
 			(layers "*.Cu" "*.Mask")
-			(remove_unused_layers yes)
-			(keep_end_layers yes)
-			(zone_layer_connections)
+			(remove_unused_layers no)
 			(net 9 "/SCL")
 			(pinfunction "Pin_5")
@@
 			(drill 1)
 			(layers "*.Cu" "*.Mask")
-			(remove_unused_layers yes)
-			(keep_end_layers yes)
-			(zone_layer_connections)
+			(remove_unused_layers no)
 			(net 6 "/INT2")
 			(pinfunction "Pin_6")
@@
 			(drill 1)
 			(layers "*.Cu" "*.Mask")
-			(remove_unused_layers yes)
-			(keep_end_layers yes)
-			(zone_layer_connections)
+			(remove_unused_layers no)
 			(net 7 "/CS")
 			(pinfunction "Pin_7")
@@
 			(drill 1)
 			(layers "*.Cu" "*.Mask")
-			(remove_unused_layers yes)
-			(keep_end_layers yes)
-			(zone_layer_connections)
+			(remove_unused_layers no)
 			(net 2 "GND")
 			(pinfunction "Pin_8")
@@
 			(drill 1)
 			(layers "*.Cu" "*.Mask")
-			(remove_unused_layers yes)
-			(keep_end_layers yes)
-			(zone_layer_connections)
+			(remove_unused_layers no)
 			(net 14 "/5V {slash} 3V3")
 			(pinfunction "Pin_9")
@@
 		)
 	)
+	(gr_text "FSYNC"
+		(at 60.382672 46.820815 -0)
+		(layer "B.SilkS")
+		(effects
+			(font
+				(size 0.85 0.85)
+				(thickness 0.15)
+			)
+			(justify right bottom mirror)
+		)
+	)
 	(gr_text "SDA"
 		(at 125.305 87.224022 0)
@@
 		)
 	)
+	(gr_text "SleepyPandas"
+		(at 72.5 25 0)
+		(layer "B.SilkS")
+		(effects
+			(font
+				(size 1 1)
+				(thickness 0.1)
+			)
+			(justify left bottom mirror)
+		)
+	)
+	(gr_text "SDA"
+		(at 60.382672 39.220815 -0)
+		(layer "B.SilkS")
+		(effects
+			(font
+				(size 0.85 0.85)
+				(thickness 0.15)
+			)
+			(justify right bottom mirror)
+		)
+	)
+	(gr_text "SCL"
+		(at 60.382672 36.720815 -0)
+		(layer "B.SilkS")
+		(effects
+			(font
+				(size 0.85 0.85)
+				(thickness 0.15)
+			)
+			(justify right bottom mirror)
+		)
+	)
 	(gr_text "CS"
 		(at 125.275 79.527447 0)
@@
 		)
 	)
+	(gr_text "INT1"
+		(at 60.382672 44.120815 -0)
+		(layer "B.SilkS")
+		(effects
+			(font
+				(size 0.85 0.85)
+				(thickness 0.15)
+			)
+			(justify right bottom mirror)
+		)
+	)
+	(gr_text "GND"
+		(at 60.352672 29.021793 -0)
+		(layer "B.SilkS")
+		(effects
+			(font
+				(size 0.85 0.85)
+				(thickness 0.15)
+			)
+			(justify right bottom mirror)
+		)
+	)
+	(gr_text "VCC"
+		(at 60.352672 26.509337 -0)
+		(layer "B.SilkS")
+		(effects
+			(font
+				(size 0.85 0.85)
+				(thickness 0.15)
+			)
+			(justify right bottom mirror)
+		)
+	)
 	(gr_text "INT2\n"
 		(at 125.305 82.124022 0)
@@
 		)
 	)
+	(gr_text "CS"
+		(at 60.352672 31.52424 -0)
+		(layer "B.SilkS")
+		(effects
+			(font
+				(size 0.85 0.85)
+				(thickness 0.15)
+			)
+			(justify right bottom mirror)
+		)
+	)
+	(gr_text "INT2\n"
+		(at 60.382672 34.120815 -0)
+		(layer "B.SilkS")
+		(effects
+			(font
+				(size 0.85 0.85)
+				(thickness 0.15)
+			)
+			(justify right bottom mirror)
+		)
+	)
 	(gr_text "INT1"
 		(at 125.305 92.124022 0)
+		(layer "B.SilkS")
+		(effects
+			(font
+				(size 0.85 0.85)
+				(thickness 0.15)
+			)
+			(justify right bottom mirror)
+		)
+	)
+	(gr_text "SD0"
+		(at 60.382672 41.720815 -0)
 		(layer "B.SilkS")
 		(effects
@@
 		)
 	)
-	(gr_text_box "Anthony Hua V1.0"
+	(gr_text_box "Anthony Hua V1.1"
 		(start 64.93125 46.490625)
 		(end 73.06875 49.009375)
