File: 0603 Parts/ICM-42670-P Breakout Board 0603.kicad_pcb (KiCad board)
At the start: 2 copper layers, 19.5 x 26.5 mm, 14 parts, among them J2 Conn_01x09_Pin, U1 ICM-42670-P, U3 MCP1700x-330xxTT

Commit message: Clean up redundant Traces / tracks
Changed lines of the file:
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@@
+	)
+	(segment
+		(start 65.252999 41.16)
+		(end 67.499999 38.913)
+		(width 0.15)
+		(layer "F.Cu")
+		(net "/SDO")
+	)
+	(segment
+		(start 58.5 41.16)
+		(end 65.252999 41.16)
+		(width 0.15)
+		(layer "F.Cu")
+		(net "/SDO")
+	)
+	(segment
+		(start 58.5 43.7)
+		(end 64.6841 43.7)
+		(width 0.15)
+		(layer "F.Cu")
+		(net "/INT1")
+	)
+	(segment
+		(start 64.6841 43.7)
+		(end 69.000001 39.384099)
+		(width 0.15)
+		(layer "F.Cu")
+		(net "/INT1")
+	)
+	(segment
+		(start 69.000001 39.384099)
+		(end 69.000001 38.913)
+		(width 0.15)
+		(layer "F.Cu")
+		(net "/INT1")
 	)
 	(segment
@@
 	)
 	(segment
-		(start 65.322904 32.927096)
-		(end 65.325 32.925)
-		(width 0.15)
-		(layer "F.Cu")
-		(net "/3V3_Clean")
-	)
-	(segment
 		(start 69.000001 36.249999)
 		(end 69.5 35.75)
@@
 		(start 72.891 39.641651)
 		(end 72.016325 40.516325)
-		(width 0.3)
-		(layer "F.Cu")
-		(net "/3V3_Clean")
-	)
-	(segment
-		(start 69.427654 34.554635)
-		(end 69.429241 34.556222)
 		(width 0.3)
 		(layer "F.Cu")
@@
 		(layer "B.Cu")
 		(net "/3V3_Clean")
-	)
-	(segment
-		(start 71.25 39.717349)
-		(end 71.257651 39.725)
-		(width 0.3)
-		(layer "F.Cu")
-		(net "GND")
 	)
 	(segment
@@
 		(layer "B.Cu")
 		(net "GND")
-	)
-	(segment
-		(start 72.127344 44.985156)
-		(end 72.175 44.9375)
-		(width 0.2)
-		(layer "F.Cu")
-		(net "Net-(D1-A)")
-	)
-	(segment
-		(start 70.263346 44.985156)
-		(end 72.127344 44.985156)
-		(width 0.2)
-		(layer "F.Cu")
-		(net "Net-(D1-A)")
-	)
-	(segment
-		(start 72.1025 45.01)
-		(end 72.175 44.9375)
-		(width 0.15)
-		(layer "F.Cu")
-		(net "Net-(D1-A)")
-	)
-	(segment
-		(start 63.175 31.5)
-		(end 64.175 30.5)
-		(width 0.15)
-		(layer "F.Cu")
-		(net "/CS")
-	)
-	(segment
-		(start 66 35.909001)
-		(end 67.2975 37.206501)
-		(width 0.15)
-		(layer "F.Cu")
-		(net "/CS")
-	)
-	(segment
-		(start 58.5 31)
-		(end 62.675 31)
-		(width 0.15)
-		(layer "F.Cu")
-		(net "/CS")
-	)
-	(segment
-		(start 66 30.75)
-		(end 66 35.909001)
-		(width 0.15)
-		(layer "F.Cu")
-		(net "/CS")
-	)
-	(segment
-		(start 65.75 30.5)
-		(end 66 30.75)
-		(width 0.15)
-		(layer "F.Cu")
-		(net "/CS")
-	)
-	(segment
-		(start 64.175 30.5)
-		(end 65.75 30.5)
-		(width 0.15)
-		(layer "F.Cu")
-		(net "/CS")
-	)
-	(segment
-		(start 62.675 31)
-		(end 63.175 31.5)
-		(width 0.15)
-		(layer "F.Cu")
-		(net "/CS")
-	)
-	(segment
-		(start 65.252999 41.16)
-		(end 67.499999 38.913)
-		(width 0.15)
-		(layer "F.Cu")
-		(net "/SDO")
-	)
-	(segment
-		(start 58.5 41.16)
-		(end 65.252999 41.16)
-		(width 0.15)
-		(layer "F.Cu")
-		(net "/SDO")
-	)
-	(segment
-		(start 58.5 43.7)
-		(end 64.6841 43.7)
-		(width 0.15)
-		(layer "F.Cu")
-		(net "/INT1")
-	)
-	(segment
-		(start 64.6841 43.7)
-		(end 69.000001 39.384099)
-		(width 0.15)
-		(layer "F.Cu")
-		(net "/INT1")
-	)
-	(segment
-		(start 69.000001 39.384099)
-		(end 69.000001 38.913)
-		(width 0.15)
-		(layer "F.Cu")
-		(net "/INT1")
 	)
 	(segment
@@
 	)
 	(segment
+		(start 63.175 31.5)
+		(end 64.175 30.5)
+		(width 0.15)
+		(layer "F.Cu")
+		(net "/CS")
+	)
+	(segment
+		(start 66 35.909001)
+		(end 67.2975 37.206501)
+		(width 0.15)
+		(layer "F.Cu")
+		(net "/CS")
+	)
+	(segment
+		(start 58.5 31)
+		(end 62.675 31)
+		(width 0.15)
+		(layer "F.Cu")
+		(net "/CS")
+	)
+	(segment
+		(start 66 30.75)
+		(end 66 35.909001)
+		(width 0.15)
+		(layer "F.Cu")
+		(net "/CS")
+	)
+	(segment
+		(start 65.75 30.5)
+		(end 66 30.75)
+		(width 0.15)
+		(layer "F.Cu")
+		(net "/CS")
+	)
+	(segment
+		(start 64.175 30.5)
+		(end 65.75 30.5)
+		(width 0.15)
+		(layer "F.Cu")
+		(net "/CS")
+	)
+	(segment
+		(start 62.675 31)
+		(end 63.175 31.5)
+		(width 0.15)
+		(layer "F.Cu")
+		(net "/CS")
+	)
+	(segment
 		(start 65.221899 36.08)
 		(end 64.505 36.08)
@@
 	)
 	(segment
+		(start 70.263346 44.985156)
+		(end 72.127344 44.985156)
+		(width 0.2)
+		(layer "F.Cu")
+		(net "Net-(D1-A)")
+	)
+	(segment
