File: Schematic PCB Design/ICM-42670-P Breakout Board 0603.kicad_sch (KiCad schematic)
At the start: 14 parts, among them J2 Conn_01x09_Pin, U1 ICM-42670-P, U3 MCP1700x-330xxTT

Commit message: Swap CS and INT2 Pins
Connections:
- net CS: now also J2.6 (Pin_6); no longer J2.7 (Pin_7)
- net INT2: now also J2.7 (Pin_7); no longer J2.6 (Pin_6)
Changed lines of the file:
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@@
 	(wire
 		(pts
-			(xy 222.25 71.12) (xy 224.79 71.12)
+			(xy 222.25 66.04) (xy 224.79 66.04)
 		)
 		(stroke
@@
 	(wire
 		(pts
-			(xy 222.25 63.5) (xy 224.79 63.5)
+			(xy 222.25 71.12) (xy 224.79 71.12)
 		)
 		(stroke
@@
 	(wire
 		(pts
+			(xy 222.25 63.5) (xy 224.79 63.5)
+		)
+		(stroke
+			(width 0)
+			(type default)
+		)
+	)
+	(wire
+		(pts
 			(xy 55.88 58.42) (xy 58.42 58.42)
 		)
@@
 	(wire
 		(pts
-			(xy 222.25 66.04) (xy 224.79 66.04)
-		)
-		(stroke
-			(width 0)
-			(type default)
-		)
-	)
-	(wire
-		(pts
 			(xy 34.29 53.34) (xy 58.42 53.34)
 		)
@@
 	)
 	(label "CS"
-		(at 222.25 63.5 180)
+		(at 222.25 66.04 180)
 		(effects
 			(font
@@
 	)
 	(label "INT2"
-		(at 222.25 66.04 180)
+		(at 222.25 63.5 180)
 		(effects
 			(font

Commit message: Changed Pin outs
Connections:
- net CS: now also J2.4 (Pin_4); no longer J2.6 (Pin_6)
- net INT2: now also J2.3 (Pin_3); no longer J2.7 (Pin_7)
- net SCL: now also J2.7 (Pin_7); no longer J2.5 (Pin_5)
- net SDA: now also J2.6 (Pin_6); no longer J2.4 (Pin_4)
- net SDO: now also J2.5 (Pin_5); no longer J2.3 (Pin_3)
Changed lines of the file:
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@@
 	(wire
 		(pts
-			(xy 196.85 50.8) (xy 196.85 48.26)
+			(xy 222.25 73.66) (xy 224.79 73.66)
 		)
 		(stroke
@@
 	(wire
 		(pts
-			(xy 186.69 48.26) (xy 186.69 58.42)
+			(xy 196.85 50.8) (xy 196.85 48.26)
 		)
 		(stroke
@@
 	(wire
 		(pts
-			(xy 55.88 55.88) (xy 58.42 55.88)
+			(xy 186.69 48.26) (xy 186.69 58.42)
 		)
 		(stroke
@@
 	(wire
 		(pts
-			(xy 29.21 53.34) (xy 34.29 53.34)
+			(xy 55.88 55.88) (xy 58.42 55.88)
 		)
 		(stroke
@@
 	(wire
 		(pts
-			(xy 41.91 58.42) (xy 43.18 58.42)
+			(xy 29.21 53.34) (xy 34.29 53.34)
 		)
 		(stroke
@@
 	(wire
 		(pts
-			(xy 154.94 55.88) (xy 157.48 55.88)
+			(xy 41.91 58.42) (xy 43.18 58.42)
 		)
 		(stroke
@@
 	(wire
 		(pts
-			(xy 154.94 48.26) (xy 163.83 48.26)
+			(xy 154.94 55.88) (xy 157.48 55.88)
 		)
 		(stroke
@@
 	(wire
 		(pts
-			(xy 222.25 66.04) (xy 224.79 66.04)
+			(xy 154.94 48.26) (xy 163.83 48.26)
 		)
 		(stroke
@@
 	(wire
 		(pts
-			(xy 222.25 71.12) (xy 224.79 71.12)
+			(xy 217.17 60.96) (xy 224.79 60.96)
 		)
 		(stroke
@@
 	(wire
 		(pts
-			(xy 217.17 60.96) (xy 224.79 60.96)
+			(xy 195.58 26.67) (xy 198.12 26.67)
 		)
 		(stroke
@@
 	(wire
 		(pts
-			(xy 195.58 26.67) (xy 198.12 26.67)
+			(xy 222.25 71.12) (xy 224.79 71.12)
 		)
 		(stroke
@@
 	(wire
 		(pts
-			(xy 222.25 73.66) (xy 224.79 73.66)
-		)
-		(stroke
-			(width 0)
-			(type default)
-		)
-	)
-	(wire
-		(pts
 			(xy 55.88 50.8) (xy 58.42 50.8)
 		)
@@
 	(wire
 		(pts
-			(xy 222.25 68.58) (xy 224.79 68.58)
+			(xy 214.63 58.42) (xy 224.79 58.42)
 		)
 		(stroke
@@
 	(wire
 		(pts
-			(xy 214.63 58.42) (xy 224.79 58.42)
+			(xy 186.69 58.42) (xy 189.23 58.42)
 		)
 		(stroke
@@
 	(wire
 		(pts
-			(xy 186.69 58.42) (xy 189.23 58.42)
+			(xy 182.88 57.15) (xy 182.88 58.42)
 		)
 		(stroke
@@
 	(wire
 		(pts
-			(xy 182.88 57.15) (xy 182.88 58.42)
+			(xy 55.88 58.42) (xy 58.42 58.42)
 		)
 		(stroke
@@
 	(wire
 		(pts
-			(xy 222.25 63.5) (xy 224.79 63.5)
+			(xy 163.83 58.42) (xy 171.45 58.42)
 		)
 		(stroke
@@
 	(wire
 		(pts
-			(xy 55.88 58.42) (xy 58.42 58.42)
+			(xy 177.8 48.26) (xy 179.07 48.26)
 		)
 		(stroke
@@
 	(wire
 		(pts
-			(xy 163.83 58.42) (xy 171.45 58.42)
+			(xy 154.94 45.72) (xy 163.83 45.72)
 		)
 		(stroke
@@
 	(wire
 		(pts
-			(xy 177.8 48.26) (xy 179.07 48.26)
+			(xy 177.8 68.58) (xy 177.8 71.12)
 		)
 		(stroke
@@
 	(wire
 		(pts
-			(xy 154.94 45.72) (xy 163.83 45.72)
+			(xy 55.88 63.5) (xy 55.88 58.42)
 		)
 		(stroke
@@
 	(wire
 		(pts
-			(xy 177.8 68.58) (xy 177.8 71.12)
+			(xy 171.45 48.26) (xy 171.45 58.42)
 		)
 		(stroke
@@
 	(wire
 		(pts
-			(xy 55.88 63.5) (xy 55.88 58.42)
+			(xy 177.8 58.42) (xy 182.88 58.42)
 		)
 		(stroke
@@
 	(wire
 		(pts
-			(xy 171.45 48.26) (xy 171.45 58.42)
+			(xy 163.83 68.58) (xy 163.83 71.12)
 		)
 		(stroke
@@
 	(wire
 		(pts
-			(xy 177.8 58.42) (xy 182.88 58.42)
+			(xy 222.25 63.5) (xy 224.79 63.5)
 		)
 		(stroke
@@
 	(wire
 		(pts
-			(xy 163.83 68.58) (xy 163.83 71.12)
+			(xy 185.42 26.67) (xy 187.96 26.67)
 		)
 		(stroke
@@
 	(wire
 		(pts
-			(xy 185.42 26.67) (xy 187.96 26.67)
+			(xy 222.25 66.04) (xy 224.79 66.04)
 		)
 		(stroke
@@
 	(wire
 		(pts
+			(xy 222.25 68.58) (xy 224.79 68.58)
+		)
+		(stroke
+			(width 0)
+			(type default)
+		)
+	)
+	(wire
+		(pts
 			(xy 50.8 58.42) (xy 55.88 58.42)
 		)
@@
 	)
 	(label "CS"
-		(at 222.25 66.04 180)
+		(at 222.25 71.12 180)
 		(effects
 			(font
@@
 	)
 	(label "INT2"
-		(at 222.25 63.5 180)
+		(at 222.25 73.66 180)
 		(effects
 			(font
@@
 	)
 	(label "SDO"
-		(at 222.25 73.66 180)
+		(at 222.25 68.58 180)
 		(effects
 			(font
@@
 	)
 	(label "SDA"
-		(at 222.25 71.12 180)
+		(at 222.25 66.04 180)
 		(effects
 			(font
@@
 	)
 	(label "SCL"
-		(at 222.25 68.58 180)
+		(at 222.25 63.5 180)
 		(effects
 			(font

Commit message: Moved around Nets for better trace routing
Connections:
- net CS: now also J2.7 (Pin_7); no longer J2.4 (Pin_4)
- net SCL: now also J2.6 (Pin_6); no longer J2.7 (Pin_7)
- net SDA: now also J2.5 (Pin_5); no longer J2.6 (Pin_6)
- net SDO: now also J2.4 (Pin_4); no longer J2.5 (Pin_5)
Changed lines of the file:
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@@
 	(wire
 		(pts
-			(xy 222.25 71.12) (xy 224.79 71.12)
+			(xy 204.47 58.42) (xy 214.63 58.42)
 		)
 		(stroke
@@
 	(wire
 		(pts
-			(xy 204.47 58.42) (xy 214.63 58.42)
+			(xy 222.25 78.74) (xy 224.79 78.74)
 		)
 		(stroke
@@
 	(wire
 		(pts
-			(xy 222.25 78.74) (xy 224.79 78.74)
+			(xy 205.74 48.26) (xy 207.01 48.26)
 		)
 		(stroke
@@
 	(wire
 		(pts
-			(xy 205.74 48.26) (xy 207.01 48.26)
+			(xy 55.88 50.8) (xy 58.42 50.8)
 		)
 		(stroke
@@
 	(wire
 		(pts
-			(xy 55.88 50.8) (xy 58.42 50.8)
+			(xy 214.63 48.26) (xy 214.63 58.42)
 		)
 		(stroke
@@
 	(wire
 		(pts
-			(xy 214.63 48.26) (xy 214.63 58.42)
+			(xy 34.29 67.31) (xy 34.29 72.39)
 		)
 		(stroke
@@
 	(wire
 		(pts
-			(xy 34.29 67.31) (xy 34.29 72.39)
+			(xy 222.25 63.5) (xy 224.79 63.5)
 		)
 		(stroke
@@
 	(wire
 		(pts
-			(xy 177.8 58.42) (xy 182.88 58.42)
+			(xy 222.25 68.58) (xy 224.79 68.58)
 		)
 		(stroke
@@
 	(wire
 		(pts
-			(xy 163.83 68.58) (xy 163.83 71.12)
+			(xy 177.8 58.42) (xy 182.88 58.42)
 		)
 		(stroke
@@
 	(wire
 		(pts
-			(xy 222.25 63.5) (xy 224.79 63.5)
+			(xy 163.83 68.58) (xy 163.83 71.12)
 		)
 		(stroke
@@
 	(wire
 		(pts
-			(xy 34.29 53.34) (xy 58.42 53.34)
+			(xy 222.25 71.12) (xy 224.79 71.12)
 		)
 		(stroke
@@
 	(wire
 		(pts
-			(xy 182.88 58.42) (xy 186.69 58.42)
+			(xy 34.29 53.34) (xy 58.42 53.34)
 		)
 		(stroke
@@
 	(wire
 		(pts
-			(xy 222.25 68.58) (xy 224.79 68.58)
+			(xy 182.88 58.42) (xy 186.69 58.42)
 		)
 		(stroke
@@
 	)
 	(label "CS"
-		(at 222.25 71.12 180)
+		(at 222.25 63.5 180)
 		(effects
 			(font
@@
 	)
 	(label "SDO"
-		(at 222.25 68.58 180)
+		(at 222.25 71.12 180)
 		(effects
 			(font
@@
 	)
 	(label "SDA"
-		(at 222.25 66.04 180)
+		(at 222.25 68.58 180)
 		(effects
 			(font
@@
 	)
 	(label "SCL"
-		(at 222.25 63.5 180)
+		(at 222.25 66.04 180)
 		(effects
 			(font

Commit message: Changed Revision to 1.3V And Changed JLCPCB part numbers
Parts:
- R1, R2, R4, R5: JLCPCB Part # C328298 -> C25804
- R3: value 120Ω -> 150 Ω; JLCPCB Part # C352482 -> C22808
Changed lines of the file:
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@@
 	(title_block
 		(title "ICM-42670-P Motion Sensor Breakout with Power Regulation")
-		(date "2026-March-26")
-		(rev "v1.2")
+		(date "2026-April-02")
+		(rev "v1.3")
 		(company "Anthony Hua / SleepPandas")
 	)
@@
 			)
 		)
-		(property "JLCPCB Part #" "C328298"
+		(property "JLCPCB Part #" "C25804"
 			(at 167.64 48.26 90)
 			(hide yes)
@@
 			)
 		)
-		(property "JLCPCB Part #" "C328298"
+		(property "JLCPCB Part #" "C25804"
 			(at 167.64 45.72 90)
 			(hide yes)
@@
 			)
 		)
-		(property "JLCPCB Part #" "C328298"
+		(property "JLCPCB Part #" "C25804"
 			(at 167.64 43.18 90)
 			(hide yes)
@@
 			)
 		)
-		(property "JLCPCB Part #" "C328298"
+		(property "JLCPCB Part #" "C25804"
 			(at 46.99 58.42 90)
 			(hide yes)
@@
 			)
 		)
-		(property "Value" "120Ω"
+		(property "Value" "150 Ω"
 			(at 201.93 22.86 90)
 			(show_name no)
@@
 			)
 		)
-		(property "JLCPCB Part #" "C352482"
+		(property "JLCPCB Part #" "C22808"
 			(at 201.93 26.67 90)
 			(hide yes)
